File: gps_interposer/gps_interposer.kicad_pcb (KiCad board)
At the start: 2 copper layers, 43 x 43.5 mm, 43 parts, among them J1 Module Connector, J2 Motherboard/Carrier Connector, J3 Ext VSYS, J4 GENERIC_3V0, J6 GENERIC_3V3, U1 SN74LVC1T45DBV, U2 SN74LVC1T45DBV, U3 RP20240-Zero, U4 SN74LVC1T45DBV, U5 SN74LVC1T45DBV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

Commit message: PCB ready.
Parts:
- removed J4: GENERIC_3V0, Connector_PinHeader_2.54mm:PinHeader_1x01_P2.54mm_Horizontal
- removed J6: GENERIC_3V3, Connector_PinHeader_2.54mm:PinHeader_1x01_P2.54mm_Horizontal
- removed JP1: TXD Direct, Connector_PinHeader_2.54mm:PinHeader_1x03_P2.54mm_Horizontal
- removed JP2: RXD Direct, Connector_PinHeader_2.54mm:PinHeader_1x03_P2.54mm_Horizontal
- removed JP4: 3V3 Zero, Connector_PinHeader_2.54mm:PinHeader_1x02_P2.54mm_Horizontal
- removed JP5: 1PPS Direct, Connector_PinHeader_2.54mm:PinHeader_1x02_P2.54mm_Horizontal
- removed R17, R18: NC, Resistor_SMD:R_0603_1608Metric_Pad0.98x0.95mm_HandSolder
- removed R19: 1K, Resistor_SMD:R_0603_1608Metric_Pad0.98x0.95mm_HandSolder
- removed U6: SN74LVC1T45DBV, Package_TO_SOT_SMD:SOT-23-6
- added C1: 100n, Capacitor_SMD:C_0603_1608Metric_Pad1.08x0.95mm_HandSolder, B.Cu at (173.5, 88.2)
- added C2: 100n, Capacitor_SMD:C_0603_1608Metric_Pad1.08x0.95mm_HandSolder, B.Cu at (197.7, 108.2)
- added C4: 100n, Capacitor_SMD:C_0603_1608Metric_Pad1.08x0.95mm_HandSolder, B.Cu at (197.7, 97.7)
- added H1: MountingHole_Pad, Kicad_Personal:MountingHole_3.7mm_3.9mm_Pad_TopBottom, F.Cu at (217.1, 77.9)
- added H2: MountingHole_Pad, Kicad_Personal:MountingHole_3.7mm_3.9mm_Pad_TopBottom, F.Cu at (217.1, 112.1)
- added H3: MountingHole_Pad, Kicad_Personal:MountingHole_3.7mm_3.9mm_Pad_TopBottom, F.Cu at (162.9, 112.1)
- added H4: MountingHole_Pad, Kicad_Personal:MountingHole_3.7mm_3.9mm_Pad_TopBottom, F.Cu at (162.9, 77.9)
- added H5: MountingHole_Pad, Kicad_Personal:MountingHole_3.7mm_3.9mm_Pad_TopBottom, F.Cu at (162.9, 69.9)
- added H6: MountingHole_Pad, Kicad_Personal:MountingHole_3.7mm_3.9mm_Pad_TopBottom, F.Cu at (217.1, 69.9)
- added H7: MountingHole_Pad, Kicad_Personal:MountingHole_3.7mm_3.9mm_Pad_TopBottom, F.Cu at (217.1, 104.1)
- added H8: MountingHole_Pad, Kicad_Personal:MountingHole_3.7mm_3.9mm_Pad_TopBottom, F.Cu at (162.9, 104.1)
- added R28: NS, Resistor_SMD:R_0603_1608Metric_Pad0.98x0.95mm_HandSolder, F.Cu at (182.7, 111.0)
- added R29: 0, Resistor_SMD:R_0603_1608Metric_Pad0.98x0.95mm_HandSolder, F.Cu at (182.6, 112.6)
- added R30: NS, Resistor_SMD:R_0603_1608Metric_Pad0.98x0.95mm_HandSolder, F.Cu at (182.6, 106.3)
- added R31: 0, Resistor_SMD:R_0603_1608Metric_Pad0.98x0.95mm_HandSolder, F.Cu at (170.0, 98.9)
- added R32: 0, Resistor_SMD:R_0603_1608Metric_Pad0.98x0.95mm_HandSolder, F.Cu at (205.0, 106.3)
- added R33: 0, Resistor_SMD:R_0603_1608Metric_Pad0.98x0.95mm_HandSolder, F.Cu at (174.2, 109.4)
- R2, R5: value NC -> NS
- moved J3 123.5 mm to (207.7, 110.7), turned to -90 degrees
- moved R2 118.3 mm to (193.7, 113.8), turned to 180 degrees
- moved R6 117.3 mm to (197.7, 111.2), turned to 0 degrees
- moved R5 115.4 mm to (197.7, 109.7), turned to 180 degrees
- moved U1 115.0 mm to (193.7, 111.2), turned to 180 degrees
- moved R13 114.7 mm to (189.3, 112.7), turned to 0 degrees
- moved R14 112.0 mm to (189.3, 110.7), turned to 0 degrees
- moved R1 111.7 mm to (193.7, 108.7), turned to 0 degrees
- moved R3 111.6 mm to (197.7, 106.7), turned to 0 degrees
- moved R4 109.7 mm to (197.7, 105.2), turned to 180 degrees
- moved U2 108.3 mm to (193.7, 106.0), turned to 180 degrees
- moved R10 104.8 mm to (193.9, 103.2), turned to 180 degrees
- moved R12 104.7 mm to (197.7, 101.2), turned to 0 degrees
- moved U3 104.2 mm to (193.7, 102.9), turned to 180 degrees
- moved R11 102.9 mm to (197.7, 99.7), turned to 180 degrees
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Routing:
- net GND: track 6.49 -> 248.7 mm, vias 0 -> 1
- net +3V0: track 6.34 -> 86.6 mm, vias 0 -> 8
- net +3.3V: track 0.00 -> 76.8 mm, vias 0 -> 8
- net /1PPS_M_3V3: track 1.70 -> 25.1 mm
- net /TXD_M: track 20.0 -> 41.2 mm, vias 1 -> 5
- net /TXD_C: track 10.8 -> 28.5 mm, vias 1 -> 2
- net /RXD_M_3V0: track 30.1 -> 13.3 mm, vias 0 -> 1
- net /TXD_C_3V0: track 30.4 -> 14.6 mm
- net Net-(U7-DIR): track 0.00 -> 15.9 mm
- net /RSVD7_C: track 3.19 -> 14.3 mm
- net Net-(U5-DIR): track 0.00 -> 9.07 mm
- net /1PPS_C: track 12.6 -> 4.34 mm, vias 0 -> 1
- net /BATT_C: track 6.59 -> 14.7 mm
- net Net-(U3-3V3): track 11.6 -> 3.45 mm
- net /ANT_BIAS_M: track 9.78 -> 2.26 mm, vias 2 -> 0
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- added copper zone on F.Cu, net +3V0
- added copper zone on B.Cu, net GND
Other:
- board size 43 x 43.5 mm -> 60.1 x 48 mm
- board text added: "GPS Interposer Tom Verbeure"

Commit message: PCB v2.
Parts:
- removed C1, C2, C4: 100n, Capacitor_SMD:C_0603_1608Metric_Pad1.08x0.95mm_HandSolder
- removed J3: Ext VSYS, Connector_PinHeader_2.54mm:PinHeader_1x02_P2.54mm_Horizontal
- removed R1, R11, R20, R27, R3, R8: NC, Resistor_SMD:R_0603_1608Metric_Pad0.98x0.95mm_HandSolder
- removed R12, R21, R4, R6, R9: 1K, Resistor_SMD:R_0603_1608Metric_Pad0.98x0.95mm_HandSolder
- removed R22, R23, R24, R25, R26, R32, R33: 0, Resistor_SMD:R_0603_1608Metric_Pad0.98x0.95mm_HandSolder
- removed R28, R30, R5: NS, Resistor_SMD:R_0603_1608Metric_Pad0.98x0.95mm_HandSolder
- removed U1, U2, U4, U5, U7: SN74LVC1T45DBV, Package_TO_SOT_SMD:SOT-23-6
- added J5: Conn_01x04_Pin, Connector_PinHeader_2.54mm:PinHeader_1x04_P2.54mm_Horizontal, F.Cu at (212.3, 110.5)
- added R17: 9k, Resistor_SMD:R_0603_1608Metric_Pad0.98x0.95mm_HandSolder, B.Cu at (189.8, 104.9)
- added R18: 9k, Resistor_SMD:R_0603_1608Metric_Pad0.98x0.95mm_HandSolder, B.Cu at (189.8, 113.3)
- added R19: 9k, Resistor_SMD:R_0603_1608Metric_Pad0.98x0.95mm_HandSolder, B.Cu at (189.8, 101.1)
- H1, H2, H3, H4, H5, H6, H7, H8: footprint Kicad_Personal:MountingHole_3.7mm_3.9mm_Pad_TopBottom -> Kicad_Personal:MountingHole_2.5mm_3.9mm_Pad_TopBottom_1
- R10, R7: value NC -> 1k
- R2: value NS -> 1k
- R29, R31: moved to B.Cu
- moved H5 54.2 mm to (217.1, 69.9)
- moved H7 54.2 mm to (162.9, 104.1)
- moved H6 34.2 mm to (217.1, 104.1)
- moved H8 34.2 mm to (162.9, 69.9)
- moved R7 17.5 mm to (189.8, 103.1), turned to 180 degrees
- moved R31 13.6 mm to (181.6, 106.1)
- moved R29 7.24 mm to (179.6, 106.0), turned to -90 degrees
- moved R10 5.61 mm to (189.8, 99.3), turned to 0 degrees
- moved R15 5.20 mm to (189.8, 97.5)
- moved R16 4.98 mm to (189.8, 95.8)
- moved R2 4.54 mm to (189.8, 111.5)
- moved R13 3.08 mm to (189.8, 109.7)
- moved R14 2.91 mm to (189.8, 107.8)
- moved U3 1.05 mm to (192.7, 102.6)
- turned J1 to -90 degrees
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Connections:
- J1 pad 10: /RSVD10_M -> /RSVD10_C
- J1 pad 4: /1PPS_M -> /1PPS_C
- J1 pad 6: /BATT_M -> /BATT_C
- J1 pad 7: /RSVD7_M -> /RSVD7_C
- J1 pad 8: /RTCM_IN_M -> /RTCM_IN_C
- J1 pad 9: /ANT_BIAS_M -> /ANT_BIAS_C
- R10 pad 1: /TXD_C_3V0 -> /TXD_C
- R14 pad 2: /TXD_M_3V3 -> /TXD_M
- R16 pad 2: /RXD_C_3V3 -> /RXD_C
- R2 pad 1: /RXD_M_3V0 -> /RXD_M_3V3
- R2 pad 2: /RXD_M_3V3 -> /RXD_M
- R7 pad 1: /1PPS_M_3V3 -> /1PPS_C
- R7 pad 2: /1PPS_M -> /1PPS_M_3V3
- U3 pad 10: unconnected-(U3-GPIO9/SPI1_CSn/I2C0_SCL/UART1_RX-Pad10) -> /RTCM_IN_C
- U3 pad 21: Net-(U3-3V3) -> +3.3V
- U3 pad 23: Net-(J3-Pin_2) -> /VSYS
Routing:
- net +3.3V: track 76.8 -> 10.7 mm, vias 8 -> 0
- net +3V0: track 86.6 -> 48.0 mm, vias 8 -> 1
- net /1PPS_M: track 26.6 -> 0.00 mm, vias 1 -> 0
- net GND: track 248.7 -> 224.2 mm, vias 1 -> 5
- net /TXD_M: track 41.2 -> 18.4 mm, vias 5 -> 1
- net /1PPS_C: track 4.34 -> 26.8 mm
- net /1PPS_M_3V3: track 25.1 -> 6.99 mm
- net Net-(U7-DIR): track 15.9 -> 0.00 mm
- net /RXD_C: track 40.8 -> 25.3 mm
- net /TXD_C_3V0: track 14.6 -> 0.00 mm, vias 1 -> 0
- net /RTCM_IN_C: track 11.6 -> 25.6 mm
- net /RXD_M_3V0: track 13.3 -> 0.00 mm, vias 1 -> 0
- net Net-(U2-DIR): track 12.9 -> 0.00 mm
- net Net-(U1-DIR): track 10.7 -> 0.00 mm, vias 2 -> 0
- net Net-(U5-DIR): track 9.07 -> 0.00 mm
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- added copper zone on B.Cu, net +3V0
- added copper zone on F.Cu, net GND
- removed copper zone on F.Cu, net +3V0
- removed copper zone on B.Cu, net GND
Other:
- board text added: "1PPS"
- board text added: "3V0"
- board text added: "3V3"
- board text added: "5V"
- board text added: "GPS Interposer v2 Tom Verbeure https://github.com/tomverbeure/gps_interposer"
- board text added: "RP2040-Zero"
- board text added: "RTCM"
- board text added: "RXD_C"
- board text added: "RXD_M"
- board text added: "TXD_C"
- board text added: "TXD_M"
- board text removed: "GPS Interposer Tom Verbeure"

Commit message: Additional connectors.
Parts:
- added J3: Conn_01x05, Connector_PinHeader_2.54mm:PinHeader_1x05_P2.54mm_Vertical_SMD_Pin1Left, F.Cu at (172.5, 111.2)
- added J4: Conn_01x04, Connector_PinHeader_2.54mm:PinHeader_1x04_P2.54mm_Horizontal, F.Cu at (173.5, 81.0)
Routing:
- net +3.3V: track 10.7 -> 74.5 mm
- net /VSYS: track 7.93 -> 69.6 mm
- net GND: track 224.2 -> 184.4 mm
- net /TXD_M: track 18.4 -> 44.6 mm
- net /RXD_M: track 28.1 -> 50.8 mm, vias 1 -> 2
- net /TXD_C: track 20.1 -> 25.7 mm, vias 2 -> 3
- net /1PPS_C: track 26.8 -> 29.7 mm, vias 1 -> 2
- net +3V0: track 48.0 -> 50.2 mm
Other:
- outline, holes or cut-outs redrawn
- board text added: "1P"
- board text added: "G"
- board text added: "RC"
- board text added: "RM"
- board text added: "TC"
- board text added: "TM"
- board text removed: "1PPS"
- board text removed: "GPS Interposer v2 Tom Verbeure https://github.com/tomverbeure/gps_interposer"
- board text removed: "RXD_C"
- board text removed: "RXD_M"
- board text removed: "TXD_C"
- board text removed: "TXD_M"
